File: hardware/controller.brd (EAGLE design)
At the start: 168 x 70 mm, 84 parts, among them IC1 MAX3232ECD, IC3 NRF24L01P-R7, IC4 TPS562231DRLR, J2 43045-0600, K1 G5V1, K2 G5V1, Q1 16M, Q2 FDN360P, Q3 FDN360P, Q4 FDN360P, U1 ATMEGA328P-AU, U2 ATMEGA328P-AU, X1 RS232, Y1 8MHz, Y2 8MHz

Commit message: move
Parts:
- moved E2 80.1 mm to (30.5, -43.2)
- moved B2 48.6 mm to (68.6, -21.6)
- moved B1 47.8 mm to (39.4, -21.6)
Connections:
- net E_LOCK: now also J2.5
- net E_UNLOCK: now also J2.6
- net GND: now also J2.2
- net N$29: now also J2.3
Routing:
- net E_LOCK: track 0.00 -> 21.2 mm
- net N$29: track 14.0 -> 35.1 mm
- net BAT: track 114.5 -> 128.1 mm
- net E_UNLOCK: track 0.00 -> 8.35 mm
Changed lines of the file:
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@@
 <?xml version="1.0" encoding="utf-8"?>
 <!DOCTYPE eagle SYSTEM "eagle.dtd">
-<eagle version="9.5.0">
+<eagle version="9.5.1">
 <drawing>
 <settings>
@@
 <text x="29.21" y="40.005" size="1.016" layer="25" font="fixed" align="center">BAT</text>
 <text x="88.011" y="9.144" size="1.016" layer="25" font="fixed" align="center">VCC</text>
-<wire x1="11.43" y1="12.7" x2="69.85" y2="12.7" width="0.3048" layer="21"/>
-<wire x1="69.85" y1="12.7" x2="69.85" y2="35.56" width="0.3048" layer="21"/>
-<wire x1="69.85" y1="35.56" x2="11.43" y2="35.56" width="0.3048" layer="21"/>
-<wire x1="11.43" y1="12.7" x2="11.43" y2="35.56" width="0.3048" layer="21"/>
 </plain>
 <attributes>
@@
 <attribute name="VALUE" x="89.535" y="8.382" size="0.0254" layer="27"/>
 </element>
-<element name="B1" library="Fidget Spinner Example" library_urn="urn:adsk.eagle:library:9489508" package="CR2032_SMT_BAT-HLD-001" package3d_urn="urn:adsk.eagle:package:9489529/2" value="" x="25.4" y="24.13" smashed="yes" rot="MR0">
-<attribute name="NAME" x="35.814" y="32.272" size="0.8128" layer="26" font="vector" ratio="18" rot="MR0"/>
-<attribute name="VALUE" x="35.814" y="15.77" size="0.4064" layer="28" font="vector" ratio="10" rot="MR0"/>
-</element>
-<element name="B2" library="Fidget Spinner Example" library_urn="urn:adsk.eagle:library:9489508" package="CR2032_SMT_BAT-HLD-001" package3d_urn="urn:adsk.eagle:package:9489529/2" value="" x="52.07" y="24.13" smashed="yes" rot="MR0">
-<attribute name="NAME" x="62.484" y="32.272" size="0.8128" layer="26" font="vector" ratio="18" rot="MR0"/>
-<attribute name="VALUE" x="62.484" y="15.77" size="0.4064" layer="28" font="vector" ratio="10" rot="MR0"/>
+<element name="B1" library="Fidget Spinner Example" library_urn="urn:adsk.eagle:library:9489508" package="CR2032_SMT_BAT-HLD-001" package3d_urn="urn:adsk.eagle:package:9489529/2" value="" x="39.37" y="-21.59" smashed="yes" rot="MR0">
+<attribute name="NAME" x="49.784" y="-13.448" size="0.8128" layer="26" font="vector" ratio="18" rot="MR0"/>
+<attribute name="VALUE" x="49.784" y="-29.95" size="0.4064" layer="28" font="vector" ratio="10" rot="MR0"/>
+</element>
+<element name="B2" library="Fidget Spinner Example" library_urn="urn:adsk.eagle:library:9489508" package="CR2032_SMT_BAT-HLD-001" package3d_urn="urn:adsk.eagle:package:9489529/2" value="" x="68.58" y="-21.59" smashed="yes" rot="MR0">
+<attribute name="NAME" x="78.994" y="-13.448" size="0.8128" layer="26" font="vector" ratio="18" rot="MR0"/>
+<attribute name="VALUE" x="78.994" y="-29.95" size="0.4064" layer="28" font="vector" ratio="10" rot="MR0"/>
 </element>
 <element name="U1" library="Microcontroller" library_urn="urn:adsk.eagle:library:14522412" package="TQFP-32" package3d_urn="urn:adsk.eagle:package:10882639/5" value="ATMEGA328P-AU" x="11.43" y="-29.21" smashed="yes">
@@
 <attribute name="VALUE" x="0" y="-29.21" size="1.27" layer="27"/>
 </element>
-<element name="E2" library="SparkFun-RF" library_urn="urn:adsk.eagle:library:531" package="TRACE_ANTENNA_2.4GHZ_15.2MM" package3d_urn="urn:adsk.eagle:package:39575/1" value="ANTENNA-GROUNDEDTRACE-15.2MM" x="64.77" y="29.21" smashed="yes" rot="R270">
-<attribute name="NAME" x="66.04" y="29.21" size="0.6096" layer="25" font="vector" ratio="20" rot="R270" align="bottom-center"/>
-<attribute name="VALUE" x="65.786" y="29.21" size="0.6096" layer="27" font="vector" ratio="20" rot="R270" align="top-center"/>
+<element name="E2" library="SparkFun-RF" library_urn="urn:adsk.eagle:library:531" package="TRACE_ANTENNA_2.4GHZ_15.2MM" package3d_urn="urn:adsk.eagle:package:39575/1" value="ANTENNA-GROUNDEDTRACE-15.2MM" x="30.48" y="-43.18" smashed="yes" rot="R270">
+<attribute name="NAME" x="31.75" y="-43.18" size="0.6096" layer="25" font="vector" ratio="20" rot="R270" align="bottom-center"/>
+<attribute name="VALUE" x="31.496" y="-43.18" size="0.6096" layer="27" font="vector" ratio="20" rot="R270" align="top-center"/>
 </element>
 <element name="J2" library="43045-0600" package="43045-0600" value="43045-0600" x="37.719" y="60.706" smashed="yes">
@@
 <contactref element="LED2" pad="C"/>
 <contactref element="TP2" pad="TP"/>
+<contactref element="J2" pad="2"/>
 </signal>
 <signal name="N$1">
@@
 <wire x1="33.02" y1="41.91" x2="34.29" y2="40.64" width="0.508" layer="1"/>
 <wire x1="34.29" y1="40.64" x2="91.44" y2="40.64" width="0.508" layer="1"/>
-<wire x1="33.02" y1="52.07" x2="33.02" y2="44.45" width="0.508" layer="1"/>
+<wire x1="33.02" y1="44.45" x2="33.02" y2="52.07" width="0.508" layer="1"/>
 <wire x1="33.02" y1="44.45" x2="33.02" y2="41.91" width="0.508" layer="1"/>
 <wire x1="17.333" y1="52.24" x2="18.984" y2="52.24" width="0.3048" layer="1"/>
@@
 <wire x1="29.21" y1="41.91" x2="29.21" y2="44.45" width="0.3048" layer="1"/>
 <contactref element="J2" pad="1"/>
-<wire x1="26.223" y1="52.24" x2="34.719" y2="65.026" width="0" layer="19" extent="1-1"/>
+<wire x1="33.02" y1="52.07" x2="33.02" y2="63.327" width="0.508" layer="1"/>
+<wire x1="33.02" y1="63.327" x2="34.719" y2="65.026" width="0.508" layer="1"/>
 </signal>
 <signal name="N$27">
@@
 <wire x1="17.78" y1="57.15" x2="21.59" y2="57.15" width="0.508" layer="16"/>
 <wire x1="21.59" y1="57.15" x2="26.67" y2="57.15" width="0.508" layer="16"/>
+<contactref element="J2" pad="3"/>
+<wire x1="26.67" y1="57.15" x2="39.37" y2="57.15" width="0.508" layer="16"/>
+<wire x1="39.37" y1="57.15" x2="40.719" y2="58.499" width="0.508" layer="16"/>
+<wire x1="40.719" y1="58.499" x2="40.719" y2="65.026" width="0.508" layer="16"/>
 </signal>
 <signal name="E_LOCK">
 <contactref element="K1" pad="10"/>
+<contactref element="J2" pad="5"/>
+<wire x1="35.1828375" y1="69.1458" x2="34.2551625" y2="69.1458" width="0.3048" layer="1"/>
+<wire x1="37.719" y1="68.026" x2="36.3026375" y2="68.026" width="0.3048" layer="1"/>
+<wire x1="36.3026375" y1="68.026" x2="35.1828375" y2="69.1458" width="0.3048" layer="1"/>
+<wire x1="34.2551625" y1="69.1458" x2="33.6893625" y2="68.58" width="0.3048" layer="1"/>
+<wire x1="19.05" y1="68.58" x2="17.78" y2="67.31" width="0.3048" layer="1"/>
+<wire x1="33.6893625" y1="68.58" x2="19.05" y2="68.58" width="0.3048" layer="1"/>
 </signal>
 <signal name="E_UNLOCK">
 <contactref element="K2" pad="10"/>
+<contactref element="J2" pad="6"/>
+<wire x1="34.719" y1="68.026" x2="27.386" y2="68.026" width="0.3048" layer="1"/>
+<wire x1="27.386" y1="68.026" x2="26.67" y2="67.31" width="0.3048" layer="1"/>
 </signal>
 <signal name="N$34">
@@
 <contactref element="U1" pad="21"/>
 <contactref element="C22" pad="2"/>
-<wire x1="25.4" y1="24.13" x2="52.07" y2="24.13" width="0" layer="19" extent="16-16"/>
-<wire x1="7.62" y1="-19.05" x2="25.4" y2="24.13" width="0" layer="19" extent="1-16"/>
+<wire x1="39.37" y1="-21.59" x2="68.58" y2="-21.59" width="0" layer="19" extent="16-16"/>
+<wire x1="7.62" y1="-19.05" x2="39.37" y2="-21.59" width="0" layer="19" extent="1-16"/>
 <wire x1="7.3" y1="-28.01" x2="7.62" y2="-19.05" width="0" layer="19" extent="1-1"/>
 <wire x1="7.3" y1="-29.61" x2="7.3" y2="-28.01" width="0" layer="19" extent="1-1"/>
@@
 <contactref element="U1" pad="6"/>
 <contactref element="U1" pad="18"/>
-<wire x1="40.64" y1="24.13" x2="63.5" y2="24.13" width="0" layer="19" extent="16-16"/>
-<wire x1="36.83" y1="24.13" x2="40.64" y2="24.13" width="0" layer="19" extent="16-16"/>
-<wire x1="13.97" y1="24.13" x2="36.83" y2="24.13" width="0" layer="19" extent="16-16"/>
-<wire x1="7.3" y1="-28.81" x2="13.97" y2="24.13" width="0" layer="19" extent="1-16"/>
+<wire x1="57.15" y1="-21.59" x2="80.01" y2="-21.59" width="0" layer="19" extent="16-16"/>
+<wire x1="50.8" y1="-21.59" x2="57.15" y2="-21.59" width="0" layer="19" extent="16-16"/>
+<wire x1="27.94" y1="-21.59" x2="50.8" y2="-21.59" width="0" layer="19" extent="16-16"/>
+<wire x1="7.3" y1="-28.81" x2="27.94" y2="-21.59" width="0" layer="19" extent="1-16"/>
 <wire x1="7.3" y1="-30.41" x2="7.3" y2="-28.81" width="0" layer="19" extent="1-1"/>
 <wire x1="15.56" y1="-31.21" x2="7.3" y2="-30.41" width="0" layer="19" extent="1-1"/>

Commit message: remote
Parts:
- removed E2: ANTENNA-GROUNDEDTRACE-15.2MM, SparkFun-RF:TRACE_ANTENNA_2.4GHZ_15.2MM
- added ANT1: ANT-2.45-CHP-T, ANT-2.45-CHP-T:ANT-2.45-CHP-T
- added C23: 0.1uF, rcl:C0805
- added C24: 1.5pF, resistor:C0805
- added C25: 1pF, resistor:C0805
- added C26: 2.2nF, resistor:C0805
- added C27: 4.7pF, resistor:C0805
- added C28: 33nF, resistor:C0805
- added C29: 10nF, resistor:C0805
- added C30: 1nF, resistor:C0805
- added C31, C32: 18p, resistor:C0805
- added IC2: NRF24L01P-R7, NRF24L01P-R7:QFN50P400X400X95-21N
- added L5: 8.2nH, rcl:L2012C
- added L6: 2.7nH, rcl:L2012C
- added L7: 3.9nH, rcl:L2012C
- added Q5: 16Mhz, crystal:HC49UP
- added R21, R23: 10K, rcl:R0805
- added R22: 22K, rcl:R0805
- added R_FTDI: TSW-106-07-G-S, con-samtec:TSW-106-XX-G-S
- added R_RESET: (no value), jumper:SJ
- added S1, S2: B3FS-1010, B3FS-1010:B3FS-1000P
- B1, B2: device Fidget Spinner Example:CR2032_SMT_BAT-HLD-001 -> fse_custom:CR2032_SMT_BAT-HLD-001
- POWER, RESET: value B3U-1000P -> B3FS-1010; device Switch:B3U-1000P -> B3FS-1010:B3FS-1000P
- moved U$5 135.8 mm to (150.0, 20.0)
- moved B2 53.5 mm to (27.0, 12.0)
- moved U1 50.1 mm to (40.0, 12.0), turned to 270 degrees
- moved C22 49.9 mm to (40.0, 4.83)
- moved R20 49.5 mm to (32.1, 18.4), turned to 90 degrees
- moved Y2 46.2 mm to (34.7, 18.4), turned to 270 degrees
- moved B1 36.3 mm to (53.0, 12.0)
- moved POWER 4.50 mm to (86.4, 35.6)
- moved RESET 2.64 mm to (98.7, 39.4), turned to 180 degrees
Connections:
- new net N$38: S1.2, U1.1
- new net N$40: S2.1, U1.32
- new net N$41: C23.2, R_FTDI.1
- new net N$42: C23.1, R21.1, R_RESET.2, U1.29
- new net N$43: IC2.13, L5.1, L7.1
- new net N$44: R_FTDI.2, U1.31
- new net N$45: R_FTDI.3, U1.30
- new net N$46: IC2.12, L5.2, L6.1
- new net N$47: C26.1, C27.1, IC2.11, L6.2
- new net N$48: C24.1, L7.2
- new net N$49: ANT1.1, C24.2, C25.2
- new net N$50: C32.2, IC2.9, Q5.1, R23.1
- new net N$51: C31.2, IC2.10, Q5.2, R23.2
- new net N$52: IC2.16, R22.1
- new net N$53: C28.1, IC2.19
- new net N$54: IC2.3, U1.17
- new net N$55: IC2.5, U1.16
- new net N$56: IC2.4, U1.15
- new net N$57: IC2.2, U1.13
- new net N$58: IC2.1, U1.12
- net BAT: now also POWER.2; no longer POWER.1
- net GND: now also RESET.2; no longer RESET.1
- net GND1: now also C25.1, C26.2, C27.2, C28.2, C29.2, C30.2, C31.1, C32.1, IC2.14, IC2.17, IC2.20, IC2.8, R22.2, R_FTDI.5, R_FTDI.6, R_RESET.1, S1.4, S2.3
- net N$33: now also POWER.4; no longer POWER.2
- net RESET: now also RESET.4; no longer RESET.2
- net VCC/2: now also C29.1, C30.1, IC2.15, IC2.18, IC2.7, R21.2, R_FTDI.4, U1.23
Routing:
- net VCC/2: track 0.00 -> 100.1 mm, vias 0 -> 3
- net N$40: track 0.00 -> 15.3 mm
- net N$51: track 0.00 -> 14.4 mm
- net N$45: track 0.00 -> 13.4 mm, vias 0 -> 1
- net N$42: track 0.00 -> 13.4 mm, vias 0 -> 2
- net N$38: track 0.00 -> 12.8 mm
- net N$47: track 0.00 -> 12.1 mm
- net N$43: track 0.00 -> 11.1 mm
- net N$44: track 0.00 -> 10.9 mm, vias 0 -> 1
- net N$50: track 0.00 -> 10.8 mm
- net N$58: track 0.00 -> 10.7 mm, vias 0 -> 2
- net N$57: track 0.00 -> 10.1 mm, vias 0 -> 2
- net N$20: track 0.00 -> 9.04 mm
- net N$55: track 0.00 -> 9.00 mm, vias 0 -> 2
- net N$54: track 0.00 -> 8.96 mm
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- added copper zone on layer 1, net GND1
- added copper zone on layer 16, net GND1
Other:
- outline, holes or cut-outs redrawn
- board text added: "FTDI"
- board text added: "github.com/ olback/car-key"
- board text removed: "github.com/olback/car-key"

Commit message: dunno
Changed lines of the file:
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@@
 <?xml version="1.0" encoding="utf-8"?>
 <!DOCTYPE eagle SYSTEM "eagle.dtd">
-<eagle version="9.5.0">
+<eagle version="9.5.2">
 <drawing>
 <settings>
@@
 <contactref element="Q3" pad="3"/>
 <wire x1="88.778" y1="26.67" x2="88.778" y2="30.099" width="0.3048" layer="1"/>
-<wire x1="88.778" y1="30.099" x2="89.578" y2="30.099" width="0.3048" layer="1"/>
 <wire x1="88.778" y1="30.099" x2="88.778" y2="32.898" width="0.3048" layer="1"/>
 <wire x1="89.19" y1="33.31" x2="90.36" y2="33.31" width="0.3048" layer="1"/>
 <wire x1="88.778" y1="32.898" x2="89.19" y2="33.31" width="0.3048" layer="1"/>
+<wire x1="89.578" y1="30.099" x2="88.778" y2="30.099" width="0.3048" layer="1"/>
 </signal>
 <signal name="N$38">
