File: hardware/controller.sch (EAGLE design)
At the start: 79 parts, among them IC1 MAX3232ECD, IC3 NRF24L01P-R7, IC4 TPS562231DRLR, J2 43045-0600, K1 G5V1, K2 G5V1, Q1 16M, Q2 FDN360P, Q3 FDN360P, Q4 FDN360P, U1 ATMEGA328P-AU, U2 ATMEGA328P-AU, X1 RS232, Y1 8MHz, Y2 8MHz

Commit message: move
Connections:
- net E_LOCK: now also J2.5
- net E_UNLOCK: now also J2.6
- net GND: now also J2.2
- net N$29: now also J2.3
Changed lines of the file:
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@@
 <?xml version="1.0" encoding="utf-8"?>
 <!DOCTYPE eagle SYSTEM "eagle.dtd">
-<eagle version="9.5.0">
+<eagle version="9.5.1">
 <drawing>
 <settings>
@@
 <attribute name="VALUE" x="195.58" y="147.32" size="1.778" layer="96" rot="R90"/>
 </instance>
-<instance part="GND8" gate="1" x="55.88" y="27.94" smashed="yes">
-<attribute name="VALUE" x="53.34" y="25.4" size="1.778" layer="96"/>
+<instance part="GND8" gate="1" x="50.8" y="20.32" smashed="yes">
+<attribute name="VALUE" x="48.26" y="17.78" size="1.778" layer="96"/>
 </instance>
 <instance part="K1" gate="1" x="86.36" y="53.34" smashed="yes">
@@
 </segment>
 <segment>
-<wire x1="53.34" y1="43.18" x2="55.88" y2="43.18" width="0.1524" layer="91"/>
-<wire x1="55.88" y1="43.18" x2="55.88" y2="30.48" width="0.1524" layer="91"/>
+<wire x1="48.26" y1="35.56" x2="50.8" y2="35.56" width="0.1524" layer="91"/>
+<wire x1="50.8" y1="35.56" x2="50.8" y2="22.86" width="0.1524" layer="91"/>
 <pinref part="GND8" gate="1" pin="GND"/>
+<pinref part="J2" gate="G$1" pin="2"/>
 </segment>
 <segment>
@@
 <junction x="106.68" y="48.26"/>
 <junction x="106.68" y="45.72"/>
+<pinref part="J2" gate="G$1" pin="3"/>
+<wire x1="27.94" y1="33.02" x2="25.4" y2="33.02" width="0.1524" layer="91"/>
+<wire x1="25.4" y1="33.02" x2="25.4" y2="25.4" width="0.1524" layer="91"/>
+<wire x1="25.4" y1="25.4" x2="53.34" y2="25.4" width="0.1524" layer="91"/>
+<wire x1="53.34" y1="25.4" x2="53.34" y2="45.72" width="0.1524" layer="91"/>
 </segment>
 </net>
 <net name="E_LOCK" class="0">
 <segment>
-<wire x1="33.02" y1="45.72" x2="30.48" y2="45.72" width="0.1524" layer="91"/>
-<wire x1="30.48" y1="45.72" x2="30.48" y2="60.96" width="0.1524" layer="91"/>
-<wire x1="30.48" y1="60.96" x2="99.06" y2="60.96" width="0.1524" layer="91"/>
+<wire x1="22.86" y1="60.96" x2="99.06" y2="60.96" width="0.1524" layer="91"/>
 <pinref part="K1" gate="2" pin="S"/>
 <wire x1="99.06" y1="60.96" x2="99.06" y2="58.42" width="0.1524" layer="91"/>
 <wire x1="99.06" y1="58.42" x2="101.6" y2="58.42" width="0.1524" layer="91"/>
+<pinref part="J2" gate="G$1" pin="5"/>
+<wire x1="27.94" y1="30.48" x2="22.86" y2="30.48" width="0.1524" layer="91"/>
+<wire x1="22.86" y1="30.48" x2="22.86" y2="60.96" width="0.1524" layer="91"/>
 </segment>
 </net>
 <net name="E_UNLOCK" class="0">
 <segment>
-<wire x1="33.02" y1="43.18" x2="27.94" y2="43.18" width="0.1524" layer="91"/>
 <wire x1="27.94" y1="43.18" x2="27.94" y2="63.5" width="0.1524" layer="91"/>
 <wire x1="27.94" y1="63.5" x2="170.18" y2="63.5" width="0.1524" layer="91"/>
@@
 <wire x1="170.18" y1="63.5" x2="170.18" y2="58.42" width="0.1524" layer="91"/>
 <wire x1="170.18" y1="58.42" x2="172.72" y2="58.42" width="0.1524" layer="91"/>
-</segment>
-</net>
+<pinref part="J2" gate="G$1" pin="6"/>
+<wire x1="48.26" y1="30.48" x2="55.88" y2="30.48" width="0.1524" layer="91"/>
+<wire x1="55.88" y1="30.48" x2="55.88" y2="43.18" width="0.1524" layer="91"/>
+<wire x1="55.88" y1="43.18" x2="27.94" y2="43.18" width="0.1524" layer="91"/>
+</segment>
+</net>

Commit message: remote
Parts:
- removed E2: ANTENNA-GROUNDEDTRACE-15.2MM, SparkFun-RF:ANTENNA-GROUNDEDTRACE-15.2MM
- added ANT1: ANT-2.45-CHP-T, ANT-2.45-CHP-T:ANT-2.45-CHP-T
- added C23: 0.1uF, rcl:C-EUC0805
- added C24: 1.5pF, resistor:C-EUC0805
- added C25: 1pF, resistor:C-EUC0805
- added C26: 2.2nF, resistor:C-EUC0805
- added C27: 4.7pF, resistor:C-EUC0805
- added C28: 33nF, resistor:C-EUC0805
- added C29: 10nF, resistor:C-EUC0805
- added C30: 1nF, resistor:C-EUC0805
- added C31, C32: 18p, resistor:C-EUC0805
- added IC2: NRF24L01P-R7, NRF24L01P-R7:NRF24L01P-R7
- added L5: 8.2nH, rcl:L-EUL2012C
- added L6: 2.7nH, rcl:L-EUL2012C
- added L7: 3.9nH, rcl:L-EUL2012C
- added Q5: 16Mhz, crystal:CRYSTALHC49UP
- added R21, R23: 10K, rcl:R-EU_R0805
- added R22: 22K, rcl:R-EU_R0805
- added R_FTDI: TSW-106-07-G-S, con-samtec:TSW-106-07-G-S
- added R_RESET: (no value), jumper:SJ
- added S1, S2: B3FS-1010, B3FS-1010:B3FS-1010
- B1, B2: device Fidget Spinner Example:BATTERYCR2032_BAT-HLD-001 -> fse_custom:BATTERYCR2032_BAT-HLD-001
- POWER, RESET: value B3U-1000P -> B3FS-1010; device Switch:B3U-1000P -> B3FS-1010:B3FS-1010
Connections:
- new net N$38: S1.COM_2, U1.PD3(PCINT19/OC2B/INT1)
- new net N$40: S2.COM_1, U1.PD2(INT0/PCINT18)
- new net N$41: C23.2, R_FTDI-1.1
- new net N$42: C23.1, R21.1, R_RESET.2, U1.(RESET/PCINT14)PC6
- new net N$43: IC2.ANT2, L5.1, L7.1
- new net N$44: R_FTDI-2.1, U1.PD1(TXD/PCINT17)
- new net N$45: R_FTDI-3.1, U1.PD0(RXD/PCINT16)
- new net N$46: IC2.ANT1, L5.2, L6.1
- new net N$47: C26.1, C27.1, IC2.VDD_PA, L6.2
- new net N$48: C24.1, L7.2
- new net N$49: ANT1.FEED, C24.2, C25.2
- new net N$50: C32.2, IC2.XC2, Q5.1, R23.1
- new net N$51: C31.2, IC2.XC1, Q5.2, R23.2
- new net N$52: IC2.IREF, R22.1
- new net N$53: C28.1, IC2.DVDD
- new net N$54: IC2.SCK, U1.(SCK/PCINT5)PB5
- new net N$55: IC2.MISO, U1.(PCINT4/MISO)PB4
- new net N$56: IC2.MOSI, U1.(PCINT3/OC2A/MOSI)PB3
- new net N$57: IC2.CSN, U1.(PCINT1/OC1A)PB1
- new net N$58: IC2.CE, U1.(PCINT0/CLKO/ICP1)PB0
- net BAT: now also POWER.COM_2; no longer POWER.1
- net GND: now also RESET.COM_2; no longer RESET.1
- net GND1: now also C25.1, C26.2, C27.2, C28.2, C29.2, C30.2, C31.1, C32.1, IC2.VSS_1, IC2.VSS_2, IC2.VSS_3, IC2.VSS_4, R22.2, R_FTDI-5.1, R_FTDI-6.1, R_RESET.1, S1.NO_2, S2.NO_1
- net N$33: now also POWER.NO_2; no longer POWER.2
- net RESET: now also RESET.NO_2; no longer RESET.2
- net VCC/2: now also C29.1, C30.1, IC2.VDD_1, IC2.VDD_2, IC2.VDD_3, R21.2, R_FTDI-4.1, U1.(ADC0/PCINT8)PC0
Other:
- note added: "TODO: Fix labels on remote Remove rulers"
- note removed: "TODO: Relay Section (relays, leds, mosfets)"
- moved on the sheet: B1, B2, C22, R20, Y2

Commit message: dunno
Other:
- note added: "TODO: Fix labels on remote Remove rulers Add resistors on signal lines"
- note removed: "TODO: Fix labels on remote Remove rulers"
Changed lines of the file:
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@@
 <?xml version="1.0" encoding="utf-8"?>
 <!DOCTYPE eagle SYSTEM "eagle.dtd">
-<eagle version="9.5.0">
+<eagle version="9.5.2">
 <drawing>
 <settings>
@@
 <text x="162.56" y="22.86" size="1.778" layer="94" align="top-left">TODO:
 Fix labels on remote
-Remove rulers</text>
+Remove rulers
+Add resistors on signal lines</text>
 </plain>
 <instances>
